File: rev_a/bus_splice.kicad_pcb (KiCad board)
At the start: 2 copper layers, 50 x 50 mm, 17 parts, among them J1 TERMINATE_JUMPER, Q1 FQP47P06, Q2 FQP47P06

Commit message: Wrapped up Rev. A
Parts:
- moved N2 40.6 mm to (116.8, 145.4), turned to 180 degrees
- moved N3 40.6 mm to (133.3, 145.4), turned to 180 degrees
- moved N4 40.6 mm to (116.8, 104.8), turned to 0 degrees
- moved N5 40.6 mm to (133.3, 104.8), turned to 0 degrees
- moved Q1 19.1 mm to (134.0, 134.6)
- moved Q2 19.1 mm to (134.0, 115.6)
- moved R2 19.1 mm to (137.8, 134.6)
- moved R3 19.1 mm to (137.8, 115.6)
- turned N1 to 270 degrees
- turned N6 to 270 degrees
Routing:
- net /LGND: track 143.4 -> 160.9 mm
- net Net-(N1-Pad6): track 49.5 -> 42.0 mm
- net /LPWR3: track 11.9 -> 9.04 mm
- net /MPWR3: track 9.04 -> 11.9 mm
- net /LPWR1: track 31.3 -> 28.8 mm
- net /MPWR1: track 28.8 -> 31.3 mm
- net /MGND: track 49.2 -> 51.4 mm
- net Net-(J1-Pad1): track 42.3 -> 43.6 mm
- net Net-(J1-Pad2): track 8.04 -> 8.56 mm
Other:
- board text added: "Bus_Splice Rev. A 2Nov2014"
- board text removed: "Bus_Splice Rev. B 2Nov2014"
