File: rev_b/bus_splice.kicad_pcb (KiCad board)
At the start: 2 copper layers, 50 x 50 mm, 17 parts, among them J1 TERMINATE_JUMPER, Q1 FQP47P06, Q2 FQP47P06

Commit message: Wrapped up Rev. B.
Parts:
- added J2: PPWR_JUMPER, Bus_Splice:Pin_Header_Straight_1x03, F.Cu at (137.8, 134.6)
- added J3: BGND_JUMPER, Bus_Splice:Pin_Header_Straight_1x03, F.Cu at (144.8, 137.2)
- added J4: LGND_JUMPER, Bus_Splice:Pin_Header_Straight_1x03, F.Cu at (144.8, 113.0)
- added J5: LPWR_JUMPER, Bus_Splice:Pin_Header_Straight_1x03, F.Cu at (137.8, 115.6)
- N1: value BUS_MASTER_HEADER -> BUS_SLAVE_HEADER
- moved R2 6.54 mm to (134.6, 140.3), turned to 0 degrees
- moved R3 6.54 mm to (134.6, 109.9), turned to 0 degrees
- moved Q1 2.54 mm to (131.4, 134.6)
- moved Q2 2.54 mm to (131.4, 115.6)
- moved G1 1.40 mm to (124.3, 113.0)
- moved N2 1.27 mm to (116.8, 146.7), turned to 0 degrees
- moved N3 1.27 mm to (133.3, 146.7), turned to 0 degrees
- moved N4 1.27 mm to (116.8, 103.5), turned to 180 degrees
- moved N5 1.27 mm to (133.3, 103.5), turned to 180 degrees
Connections:
- net /MPWR1 renamed /BPWR1
- net /MPWR2 renamed /BPWR2
- H1 pad 1: /LGND -> (no net)
- H2 pad 1: /LGND -> (no net)
- H3 pad 1: /LGND -> (no net)
- H4 pad 1: /LGND -> (no net)
- N1 pad 1: (no net) -> /LPWR0
- N1 pad 10: (no net) -> /BPWR0
- N1 pad 2: (no net) -> /LPWR0
- N1 pad 3: (no net) -> /LGND0
- N1 pad 4: (no net) -> /LGND0
- N1 pad 7: (no net) -> /BGND0
- N1 pad 8: (no net) -> /BGND0
- N1 pad 9: (no net) -> /BPWR0
- N2 pad 1: /MGND -> /BGND1
- N3 pad 1: /MGND -> /BGND1
- N4 pad 1: /LGND -> /LGND1
- N5 pad 1: /LGND -> /LGND1
- N6 pad 1: /LPWR3 -> /LPWR4
- N6 pad 10: /MPWR3 -> /BPWR4
- N6 pad 2: /LPWR3 -> /LPWR4
- N6 pad 3: /LGND -> /LGND2
- N6 pad 4: /LGND -> /LGND2
- N6 pad 7: /MGND -> /BGND2
- N6 pad 8: /MGND -> /BGND2
- N6 pad 9: /MPWR3 -> /BPWR4
- Q1 pad G: /MGND -> /BGND1
- Q2 pad G: /LGND -> /LGND1
- R2 pad 2: /MPWR3 -> /BPWR3
Routing:
- net /LGND: track 160.9 -> 0.00 mm
- net /LGND0: track 0.00 -> 72.0 mm, vias 0 -> 1
- net /BGND0: track 0.00 -> 65.3 mm
- net /LPWR0: track 0.00 -> 51.9 mm
- net /MGND: track 51.4 -> 0.00 mm
- net /BGND1: track 0.00 -> 49.4 mm
- net /LGND1: track 0.00 -> 47.5 mm
- net /BPWR0: track 0.00 -> 37.7 mm
- net /LGND2: track 0.00 -> 14.9 mm
- net /BGND2: track 0.00 -> 14.2 mm
- net /MPWR3: track 11.9 -> 0.00 mm
- net /LPWR4: track 0.00 -> 10.1 mm
- net /BPWR4: track 0.00 -> 10.1 mm
- net /BPWR2: track 3.82 -> 11.7 mm
- net /LPWR3: track 9.04 -> 3.46 mm
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Other:
- board text added: "BLK"
- board text added: "BUS"
- board text added: "BUS_SPLICE REV. B 26JAN2015"
- board text added: "BUS_SPLICE REV. B 26JAN2015 (C) 20015 GRAMLICH"
- board text added: "TERM"
- board text removed: "Bus Splice Rev. A 2Nov2014 (c) Gramlich"
- board text removed: "Bus_Splice Rev. A 2Nov2014"
- board text removed: "Term"
