File: rev_b/bus_splice.sch (KiCad schematic (older format))
At the start: 17 parts, among them J1 TERMINATE_JUMPER, Q1 FQP47P06, Q2 FQP47P06

Commit message: Wrapped up Rev. B.
Parts:
- removed N1: BUS_MASTER_HEADER, Bus_Splice:Pin_Header_Straight_2x05_Shrouded, symbol BUS_MASTER_HEADER
- added J2: PPWR_JUMPER, Bus_Splice:Pin_Header_Straight_1x03, symbol PWR_JUMPER
- added J3: BGND_JUMPER, Bus_Splice:Pin_Header_Straight_1x03, symbol PWR_JUMPER
- added J4: LGND_JUMPER, Bus_Splice:Pin_Header_Straight_1x03, symbol PWR_JUMPER
- added J5: LPWR_JUMPER, Bus_Splice:Pin_Header_Straight_1x03, symbol PWR_JUMPER
- added N1: BUS_SLAVE_HEADER, Bus_Splice:Pin_Header_Straight_2x05_Shrouded, symbol BUS_SLAVE_HEADER
- N6: footprint Bus_Splice:Pin_Header_Straight_2x05_Shrouded -> ~
Connections:
- net LPWR3: now also J5.3 (BLK); no longer N6.1 (LPWR1), N6.2 (LPWR2)
- net at J1.1 (ON), N6.5 (CANH): now also N1.5 (CANH)
- net at N6.6 (CANL), R1.2: now also N1.6 (CANL)
- removed net LGND: H1.1 (GND), H2.1 (GND), H3.1 (GND), H4.1 (GND), N4.1 (-), N5.1 (-), N6.3 (LGND1), N6.4 (LGND2), Q2.G
- net MGND renamed BGND1
- net BGND1: now also J3.3 (BLK); no longer N6.7 (BGND1), N6.8 (BGND2)
- net MPWR1 renamed BPWR1
- net MPWR2 renamed BPWR2
- net MPWR3 renamed BPWR4
- net BPWR4: now also J2.2 (OUT); no longer R2.2
- new net BGND0: J3.1 (BUS), N1.7 (BGND1), N1.8 (BGND2)
- new net BGND2: J3.2 (OUT), N6.7 (BGND1), N6.8 (BGND2)
- new net BPWR0: J2.1 (BUS), N1.10 (BPWR2), N1.9 (BPWR1)
- new net BPWR3: J2.3 (BLK), R2.2
- new net LGND0: J4.1 (BUS), N1.3 (LGND1), N1.4 (LGND2)
- new net LGND1: J4.3 (BLK), N4.1 (-), N5.1 (-), Q2.G
- new net LGND2: J4.2 (OUT), N6.3 (LGND1), N6.4 (LGND2)
- new net LPWR0: J5.1 (BUS), N1.1 (LPWR1), N1.2 (LPWR2)
- new net LPWR4: J5.2 (OUT), N6.1 (LPWR1), N6.2 (LPWR2)
- no-connect marks 9 -> 5
Other:
- moved on the sheet: G1, H1, H2, H3, H4, Q1, Q2, R2, R3
